Commit message: 뭔진 모르겠지만 조금 더 나아진 버전

File: src/arm_v3/urdf/arm_v3.urdf (robot description, URDF)
Before this commit: robot arm_v3, 9 links, 8 joints
Joints:
- joint Joint6: axis 1 0 0 -> (none); limit lower=0 upper=0.054 effort=30 velocity=4 -> (none); mimic joint=Joint7 multiplier=1 offset=0 -> (none); type prismatic -> fixed
- joint Joint7: axis 1 0 0 -> (none); limit lower=0 upper=0.054 effort=30 velocity=1 -> (none); type prismatic -> fixed

File: src/arm_v3_config/config/arm_v3.ros2_control.xacro (robot description, xacro)
@@ -43,11 +43,4 @@
                 <state_interface name="velocity"/>
             </joint>
-            <joint name="Joint7">
-                <command_interface name="position"/>
-                <state_interface name="position">
-                  <param name="initial_value">${initial_positions['Joint7']}</param>
-                </state_interface>
-                <state_interface name="velocity"/>
-            </joint>
         </ros2_control>
     </xacro:macro>
